File: esp32_Devkit_C_GRBL.sch (KiCad schematic (older format))
At the start: 49 parts, among them J1 Emergency Stop, J10 x - axis, J11 Outputs, J12 Micro_SD_Card_Adater, J13 Probe, J14 Buttons, J2 Power Supply, J3 Y1 Limit, J4 X Limit, J5 Y2 Limit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

Commit message: v0
Parts:
- C1, C2: footprint Capacitor_THT:CP_Axial_L11.0mm_D5.0mm_P18.00mm_Horizontal -> Capacitor_THT:CP_Radial_D8.0mm_P3.50mm
- C3, C4, C5, C6, C7: footprint Capacitor_THT:C_Disc_D6.0mm_W4.4mm_P5.00mm -> Capacitor_THT:C_Disc_D3.0mm_W1.6mm_P2.50mm
- D1: footprint Diode_SMD:D_2512_6332Metric -> Diode_SMD:D_SMB
- D2: footprint Diode_THT:D_A-405_P12.70mm_Horizontal -> Package_TO_SOT_SMD:TO-277B
- D3, D4, D6: footprint Diode_THT:D_A-405_P10.16mm_Horizontal -> Diode_SMD:D_SOD-123
- D5: value D -> GS1000FL; footprint Diode_THT:D_A-405_P10.16mm_Horizontal -> Diode_SMD:D_SOD-123
- J1, J2: footprint Connector_Phoenix_MC_HighVoltage:PhoenixContact_MCV_1,5_2-G-5.08_1x02_P5.08mm_Vertical -> Connector_Phoenix_GMSTB:PhoenixContact_GMSTBA_2,5_2-G-7,62_1x02_P7.62mm_Horizontal
- J10, J7, J8, J9: footprint Connector_Phoenix_MSTB:PhoenixContact_MSTBA_2,5_6-G-5,08_1x06_P5.08mm_Horizontal -> Connector_Phoenix_MSTB:PhoenixContact_MSTBA_2,5_4-G-5,08_1x04_P5.08mm_Horizontal; symbol Connector:Screw_Terminal_01x06 -> Connector:Screw_Terminal_01x04
- J12: footprint (none) -> Connector_PinHeader_2.54mm:PinHeader_1x06_P2.54mm_Vertical
- J13: footprint (none) -> Connector_Phoenix_MSTB:PhoenixContact_MSTBA_2,5_2-G-5,08_1x02_P5.08mm_Horizontal
- SW1: value Canel -> Cancel; footprint Button_Switch_THT:SW_PUSH_6mm -> Button_Switch_SMD:SW_Push_1P1T_NO_6x6mm_H9.5mm
- SW2: footprint Button_Switch_THT:SW_PUSH_6mm -> Button_Switch_SMD:SW_Push_1P1T_NO_6x6mm_H9.5mm
- SW3: value SW_Push -> Pause; footprint Button_Switch_THT:SW_PUSH_6mm -> Button_Switch_SMD:SW_Push_1P1T_NO_6x6mm_H9.5mm
- U5: footprint (none) -> Package_TO_SOT_THT:TO-220F-3_Vertical
Connections:
- net labels added: ESP32DevKitCGRBLCNC, GPIO_NUM_02
- net labels removed: 12VDC
- wire segments 252 -> 236
